File: Rosies Board.kicad_pcb (KiCad board)
At the start: 2 copper layers, 209.6 x 76.2 mm, 91 parts

Commit message: update silks
Parts:
- removed the G*** at (133.4, 54.8) (x2)
- added G***: LOGO, Eleven:eleven art 1, B.Cu at (133.4, 54.8)
- added G***: LOGO, Eleven:eleven art 1, F.Cu at (133.4, 54.8)
